File: usbconn.kicad_sch (KiCad schematic)
At the start: 3 parts, among them J3 USB_C_Receptacle_PowerOnly_6P

Commit message: cleanup
Other:
- note added: "Pull-downs to USB for UFP operation"
Changed lines of the file:
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@@
 	(generator_version "9.0")
 	(paper "A4")
+	(text "Pull-downs to USB\nfor UFP operation"
+		(exclude_from_sim no)
+		(at 182.118 96.012 0)
+		(effects
+			(font
+				(size 1.27 1.27)
+			)
+		)
+	)
 	(junction
 		(at 149.86 91.44)
