File: _autosave-gameboy.kicad_pcb (KiCad board)
At the start: 4 copper layers, 90 x 125 mm, 102 parts, among them J1 SM03B-SRSS-TB, J2 FPC-05F-12PH20, J3 Conn_01x02, J4 Conn_01x02, J5 Conn_01x02, J6 SD_Card_Receptacle, J7 USB_C_Receptacle_USB2.0_16P, Q1 SS8050, Q2 AO3401A, Q3 SS8050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

Commit message: whole bunch of layout done
Parts:
- moved R18 156.6 mm to (69.1, 192.0)
- moved C23 154.7 mm to (73.1, 189.0), turned to 90 degrees
- moved C26 152.6 mm to (101.0, 187.0), turned to -90 degrees
- moved R19 151.9 mm to (75.0, 189.0), turned to 90 degrees
- moved R21 150.7 mm to (99.0, 187.0), turned to 90 degrees
- moved SW8 149.7 mm to (84.2, 185.5), turned to -90 degrees
- moved R20 148.3 mm to (96.0, 183.0), turned to 90 degrees
- moved Q2 147.9 mm to (75.1, 185.0)
- moved L2 147.9 mm to (91.0, 189.0)
- moved R22 147.7 mm to (97.0, 187.0), turned to 90 degrees
- moved C25 144.6 mm to (89.1, 180.0)
- moved C24 144.2 mm to (72.1, 181.0), turned to 90 degrees
- moved C28 138.7 mm to (143.4, 150.0), turned to 90 degrees
- moved R16 136.4 mm to (70.1, 181.0), turned to -90 degrees
- moved D1 136.1 mm to (70.1, 178.0), turned to 90 degrees
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Connections:
- net +5V renamed VDC
Routing:
- net GND: track 0.00 -> 151.2 mm, vias 0 -> 16
- net /Power/USB_VBUS: track 0.00 -> 60.0 mm
- net +3V3: track 0.00 -> 27.2 mm, vias 0 -> 7
- net VDC: track 0.00 -> 17.4 mm
- net Net-(J6-DAT2): track 0.00 -> 15.4 mm
- net /MCU/SD_SS: track 0.00 -> 13.5 mm
- net +3.3V: track 0.00 -> 11.8 mm
- net /MCU/SD_MOSI: track 0.00 -> 11.6 mm
- net Net-(D3-K): track 0.00 -> 11.0 mm
- net /Buttons/BTN_B: track 0.00 -> 9.92 mm
- net /Buttons/BTN_UP: track 0.00 -> 9.82 mm
- net /Buttons/BTN_LEFT: track 0.00 -> 9.82 mm
- net /Buttons/BTN_DOWN: track 0.00 -> 9.82 mm
- net /Buttons/BTN_A: track 0.00 -> 9.73 mm
- net Net-(J7-CC1): track 0.00 -> 8.73 mm
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- added copper zone on B.Cu, net +3V3
- added copper zone on F.Cu, net +3V3
- added copper zone on In1.Cu, net GND
- added copper zone on In2.Cu, net GND
Other:
- outline, holes or cut-outs redrawn
