File: usb.kicad_sch (KiCad schematic)
At the start: 4 parts, among them J7 USB_C_Receptacle_USB2.0_16P, U6 USBLC6-2SC6

Commit message: whole bunch of layout done
Other:
- moved on the sheet: R23, R24, U6
