File: buttons.kicad_sch (KiCad schematic)
At the start: 18 parts, among them SW10 SW_Push, SW3 SW_Push, SW4 SW_Push, SW5 SW_Push, SW6 SW_Push, SW7 SW_Push

Commit message: update components
Parts:
- C19, C20, C21, C22, C36, C37: LCSC (none) -> C52923; Manufacturer FH -> Samsung Electro-Mechanics; Manufacturer Part Number 0603CG8R0C500NT -> CL05A105KA5NQNC
Changed lines of the file:
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@@
 			)
 		)
-		(property "LCSC" ""
+		(property "LCSC" "C52923"
 			(at 87.63 138.43 0)
 			(hide yes)
@@
 			)
 		)
-		(property "Manufacturer" "FH"
+		(property "Manufacturer" "Samsung Electro-Mechanics"
 			(at 87.63 138.43 0)
 			(hide yes)
@@
 			)
 		)
-		(property "Manufacturer Part Number" "0603CG8R0C500NT"
+		(property "Manufacturer Part Number" "CL05A105KA5NQNC"
 			(at 87.63 138.43 0)
 			(hide yes)
@@
 			)
 		)
-		(property "LCSC" ""
+		(property "LCSC" "C52923"
 			(at 123.19 104.14 0)
 			(hide yes)
@@
 			)
 		)
-		(property "Manufacturer" "FH"
+		(property "Manufacturer" "Samsung Electro-Mechanics"
 			(at 123.19 104.14 0)
 			(hide yes)
@@
 			)
 		)
-		(property "Manufacturer Part Number" "0603CG8R0C500NT"
+		(property "Manufacturer Part Number" "CL05A105KA5NQNC"
 			(at 123.19 104.14 0)
 			(hide yes)
@@
 			)
 		)
-		(property "LCSC" ""
+		(property "LCSC" "C52923"
 			(at 53.34 104.14 0)
 			(hide yes)
@@
 			)
 		)
-		(property "Manufacturer" "FH"
+		(property "Manufacturer" "Samsung Electro-Mechanics"
 			(at 53.34 104.14 0)
 			(hide yes)
@@
 			)
 		)
-		(property "Manufacturer Part Number" "0603CG8R0C500NT"
+		(property "Manufacturer Part Number" "CL05A105KA5NQNC"
 			(at 53.34 104.14 0)
 			(hide yes)
@@
 			)
 		)
-		(property "LCSC" ""
+		(property "LCSC" "C52923"
 			(at 232.41 85.09 0)
 			(hide yes)
@@
 			)
 		)
-		(property "Manufacturer" "FH"
+		(property "Manufacturer" "Samsung Electro-Mechanics"
 			(at 232.41 85.09 0)
 			(hide yes)
@@
 			)
 		)
-		(property "Manufacturer Part Number" "0603CG8R0C500NT"
+		(property "Manufacturer Part Number" "CL05A105KA5NQNC"
 			(at 232.41 85.09 0)
 			(hide yes)
@@
 			)
 		)
-		(property "LCSC" ""
+		(property "LCSC" "C52923"
 			(at 203.2 134.62 0)
 			(hide yes)
@@
 			)
 		)
-		(property "Manufacturer" "FH"
+		(property "Manufacturer" "Samsung Electro-Mechanics"
 			(at 203.2 134.62 0)
 			(hide yes)
@@
 			)
 		)
-		(property "Manufacturer Part Number" "0603CG8R0C500NT"
+		(property "Manufacturer Part Number" "CL05A105KA5NQNC"
 			(at 203.2 134.62 0)
 			(hide yes)
@@
 			)
 		)
-		(property "LCSC" ""
+		(property "LCSC" "C52923"
 			(at 88.9 71.12 0)
 			(hide yes)
@@
 			)
 		)
-		(property "Manufacturer" "FH"
+		(property "Manufacturer" "Samsung Electro-Mechanics"
 			(at 88.9 71.12 0)
 			(hide yes)
@@
 			)
 		)
-		(property "Manufacturer Part Number" "0603CG8R0C500NT"
+		(property "Manufacturer Part Number" "CL05A105KA5NQNC"
 			(at 88.9 71.12 0)
 			(hide yes)
