File: vibration.kicad_sch (KiCad schematic)
At the start: 9 parts, among them J5 Conn_01x02, Q3 SS8050

Commit message: update components
Parts:
- C34: LCSC (none) -> C52923; Manufacturer (none) -> Samsung Electro-Mechanics; Manufacturer Part Number (none) -> CL05A105KA5NQNC
- D4: value D -> B340A
Changed lines of the file:
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@@
 			)
 		)
-		(property "LCSC" ""
+		(property "LCSC" "C52923"
 			(at 119.38 74.93 0)
 			(hide yes)
@@
 			)
 		)
-	)
+		(property "Manufacturer" "Samsung Electro-Mechanics"
+			(at 119.38 74.93 0)
+			(hide yes)
+			(effects
+				(font
+					(size 1.27 1.27)
+				)
+			)
+		)
+		(property "Manufacturer Part Number" "CL05A105KA5NQNC"
+			(at 119.38 74.93 0)
+			(hide yes)
+			(effects
+				(font
+					(size 1.27 1.27)
+				)
+			)
+		))
 	(symbol
 		(lib_id "power:+3V3")
@@
 			)
 		)
-		(property "Value" "D"
+		(property "Value" "B340A"
 			(at 134.62 75.8824 90)
 			(show_name no)
